Commit message: feat(rakuda): real masses, and a current path that reaches the right motor
Everything in the Rakuda-2 plan except the gravity compensation itself, which
is being done on its own branch. P0, P1, P2, and the half of P5 that is not
about gravity.

P0 -- the current output was signed wrong. `command_torques_nm` converts Nm to
amperes in *joint* coordinates and handed them straight to
`write_goal_current_a`, which writes in the motor's own positive direction and
documents that it applies no joint sign. On a `direction = -1` joint that drives
the arm backwards under a command that reads correctly at every level above the
bus. The regression test went in first and failed as `assert 100 == -100`.

The same path now also enforces what it claimed to: the effective ceiling is the
lower of the calibrated and the configured limit, `max_current_rate_a_s` bounds
how fast a command may change, measured against real elapsed time rather than a
nominal period, and the ceiling wins over the rate so that lowering a limit takes
effect immediately. The slew reference is cleared where the hardware actually
changes -- a mode change resets GOAL_CURRENT, a stop ends the command -- and
deliberately *not* on a new lease, where the motor is still holding what the
previous generation wrote. Saturation is recorded rather than swallowed, and
`last_current_command` keeps joint amperes, motor amperes and raw counts side by
side, which is where a sign or a unit error shows.

P5 (not the gravity parts) -- reading a motor is not permission to write to it.
ArmServo takes `command_motor_names` alongside `motor_names`, enforces that the
command set is inside the read set, and reports operating modes per motor rather
than one for the port. `None` and `[]` now mean different things: the old
`motor_names or joint_map.motor_names` turned an explicit empty list into every
motor on the bus.

P1 -- the committed model weighed 2.07 grams, because the CAD export carried
volumes where masses belong. The density-corrected re-export is now imported by
`scripts/update_rakuda_inertials.py`: 7.8828710378 kg across 137 changed links,
in all three URDFs. It moves `<inertial>` blocks and nothing else, after checking
that both files describe the same machine -- links, joints, types, parents, axes,
origins, limits, mesh references and scales -- because the new export has no
collision geometry and copying it over the three would have deleted 274
`<collision>` elements. The edit is textual so the diff stays readable, and is
verified by re-parsing: 137 mass lines, 137 inertia lines and 5 origin lines that
differ in the last digits of a ~1e-16 centre-of-mass component. Forward
kinematics and frame Jacobians are bit-identical before and after, as they must
be.

P2 -- the audit conflated two questions. `usable_for_dynamics` required every
link to declare an inertial, which the static root never will, so it was False
whatever the masses said. It is now `numerically_consistent` -- plausible total,
no massless *parts* below a joint, every inertia tensor a possible rigid body --
with `hardware_validated` as a separate field that no arithmetic can set. A link
with no geometry is a coordinate frame and weighs nothing legitimately; a link
that draws something and weighs nothing is a hole. Telling them apart
structurally beats guessing from names: the Rakuda has 12 massless moving links
and none of them draws geometry. Per-joint subtree masses are reported too, which
is what keeps the 5.6 kg base plate from being read as load on the arms -- the
torso carries 1.99 kg.

The principal-moment check needed eigenvalues of a symmetric 3x3, written out in
closed form rather than pulled from NumPy so the module keeps its promise of
running on a checkout with no extras installed; a test holds it against
`numpy.linalg.eigvalsh` over 200 random tensors.

Status: verified in code and against the committed model. Nothing here has been
checked on the machine, and the audit now says so out loud.

Co-Authored-By: Claude Opus 5 (1M context) <noreply@anthropic.com>

File: src/robopy/models/rakuda/assembly_2/urdf/assembly_2.urdf (robot description, URDF)
Before this commit: robot assembly_2, 153 links, 152 joints
Links:
- link _5シリーズ2列_nfs5_2040_297_1___nfs5_2040_910: mass 9.57636e-05 -> 0.258562
- link _ゴム足Φ24x10_c_30_rk_24_black_1__none_1: mass 3.25901e-06 -> 0.00358491
- link axk1106_1___axk1106: mass 1.52808e-06 -> 0.00168089
- link axk1106_1___axk1106_1: mass 1.52808e-06 -> 0.00412582
- link axk1106_1___axk1106_2: mass 1.52808e-06 -> 0.00412582
- link base_plate_03jk_rakuda_1__ソリッド1: mass 0.000712823 -> 5.59566
- link cable_guide_fr12_hinge_head_r4_1__ソリッド1: mass 2.66493e-06 -> 0.00280351
- link elbow_cover_right: mass 1.90245e-05 -> 0.0200138
- link fr12_h104_1__ソリッド1: mass 4.31461e-06 -> 0.0116495
- link fr12_h104_1__ソリッド1_1: mass 4.31461e-06 -> 0.0116495
- link fr12_h104_1__ソリッド1_2: mass 4.31461e-06 -> 0.0116495
- link fr12_h104_1__ソリッド1_3: mass 4.31461e-06 -> 0.0116495
- link fr12_h104_1__ソリッド1_4: mass 4.31461e-06 -> 0.0116495
- link fr12_s101_1__ソリッド1: mass 3.17353e-06 -> 0.00856853
- link fr12_s101_1__ソリッド1_1: mass 3.17353e-06 -> 0.00856853
- link fr12_s102_1__ソリッド1: mass 2.0777e-06 -> 0.00560978
- link fr12_s102_1__ソリッド1_1: mass 2.0777e-06 -> 0.00560978
- link fr13_h101_1__ソリッド1: mass 6.02982e-06 -> 0.0162805
- link fr13_h101_1__ソリッド1_1: mass 6.02982e-06 -> 0.0162805
- link hn12_i101_1__ソリッド1: mass 5.41761e-07 -> 0.00146275
- link hn12_i101_1__ソリッド1_1: mass 5.41761e-07 -> 0.00146275
- link hn12_i101_1__ソリッド1_2: mass 5.41761e-07 -> 0.00146275
- link hn12_i101_1__ソリッド1_3: mass 5.41761e-07 -> 0.00146275
- link hn12_i101_1__ソリッド1_4: mass 5.41761e-07 -> 0.00146275
- link hn12_n101_1__ソリッド1: mass 5.8065e-07 -> 0.00156776
- link hn12_n101_1__ソリッド1_1: mass 5.8065e-07 -> 0.00156776
- link hn12_n101_1__ソリッド1_2: mass 5.8065e-07 -> 0.00156776
- link hn12_n101_1__ソリッド1_3: mass 5.8065e-07 -> 0.00156776
- link hn12_n101_1__ソリッド1_4: mass 5.8065e-07 -> 0.00156776
- link hn12_n101_1__ソリッド1_5: mass 5.8065e-07 -> 0.00156776
- link hn12_n101_1__ソリッド1_6: mass 5.8065e-07 -> 0.00156776
- link hn12_n101_1__ソリッド1_7: mass 5.8065e-07 -> 0.00156776
- link hn12_n101_1__ソリッド1_8: mass 5.8065e-07 -> 0.00156776
- link hn12_n101_1__ソリッド1_9: mass 5.8065e-07 -> 0.00156776
- link hn13_c101_1__ソリッド1: mass 1.76909e-06 -> 0.00477655
- link hn13_c101_1__ソリッド1_1: mass 1.76909e-06 -> 0.00477655
- link hn13_c101_1__ソリッド1_2: mass 1.76909e-06 -> 0.00477655
- link hn13_i101_1__ソリッド1: mass 1.17425e-06 -> 0.00317047
- link hn13_i101_1__ソリッド1_1: mass 1.17425e-06 -> 0.00317047
- link hn13_n101_1__ソリッド1: mass 1.22568e-06 -> 0.00330934
- link hn13_n101_1__ソリッド1_1: mass 1.22568e-06 -> 0.00330934
- link igus_jfm_1113_05_1__1: mass 3.09557e-07 -> 0.000835805
- link igus_jfm_1113_05_1__1_1: mass 3.09557e-07 -> 0.000835805
- link igus_jfm_1113_05_1__1_2: mass 3.09557e-07 -> 0.000835805
- link igus_jfm_1113_05_1__1_3: mass 3.09557e-07 -> 0.000835805
- link intel_realsense_depth_camera_d435_1__ソリッド1_1: mass 3.65256e-05 -> 0.0465255
- link rakuda29_joint_upper_arm_r1_1__ソリッド1: mass 5.54227e-06 -> 0.00583046
- link rakuda29_joint_upper_arm_r1_1__ソリッド1_1: mass 5.54227e-06 -> 0.00583046
- link rakuda2_r3_waist_base_1__ソリッド1: mass 2.8514e-05 -> 0.0299967
- link rakuda34_r2__spacer_axk1160_waist_ring_r1_1__ソリッド1: mass 2.61695e-07 -> 0.000287864
- link rakuda34_r2__spacer_axk1160_waist_ring_r1_1__ソリッド1_1: mass 2.61695e-07 -> 0.000287864
- link rakuda_r3__arm_cover_elbow_r1_1__ソリッド1: mass 1.94674e-05 -> 0.0204797
- link rakuda_r3__arm_cover_upperarm_side_1__ソリッド1: mass 2.58744e-05 -> 0.0272199
- link rakuda_r3__arm_cover_upperarm_side_1__ソリッド1_1: mass 2.58744e-05 -> 0.0272199
- link rakuda_r3__arm_joint_upper_arm_back_1__ソリッド2: mass 4.29668e-06 -> 0.00452011
- link rakuda_r3__arm_joint_upper_arm_back_1__ソリッド2_1: mass 4.29668e-06 -> 0.00452011
- link rakuda_r3__base_cable_guide_d435usb_r1_1__ソリッド1: mass 3.18899e-06 -> 0.00335482
- link rakuda_r3__chest_cover_r1_1__ソリッド1: mass 1.28949e-05 -> 0.0135654
- link rakuda_r3__head_cable_guide_d435usb_1__ソリッド1: mass 4.08926e-07 -> 0.00043019
- link rakuda_r3__head_cover_front_1__ソリッド1: mass 1.06876e-05 -> 0.0112433
- link rakuda_r3__head_mount_d435_1__ソリッド1: mass 1.89546e-05 -> 0.0199402
- link rakuda_r3__neck_cable_guide2head_base_1__ソリッド1: mass 1.04854e-05 -> 0.0110306
- link rakuda_r3__neck_cover_r4_1__ソリッド1: mass 1.89252e-05 -> 0.0199093
- link rakuda_r3__plate_waist_x540_r8_1__ソリッド1: mass 9.67876e-05 -> 0.101821
- link rakuda_r3__shoulder_base_hinge_1__ソリッド1: mass 1.4263e-05 -> 0.0150046
- link rakuda_r3__shoulder_base_hinge_1__ソリッド1_1: mass 1.4263e-05 -> 0.0150046
- link rakuda_r3__shoulder_hinge_cover_1__ソリッド1: mass 7.08032e-06 -> 0.00744849
- link rakuda_r3__shoulder_hinge_cover_1__ソリッド1_2: mass 7.08032e-06 -> 0.00744849
- link rakuda_r3__spacer_axk1160_waist_r2_1__ソリッド1: mass 5.47367e-06 -> 0.0057583
- link rakuda_r3__upper_arm_cover_inside_l_1__ソリッド1: mass 6.71233e-06 -> 0.00706138
- link rakuda_r3__upper_arm_cover_inside_l_r1_1__ソリッド1: mass 6.89641e-06 -> 0.00725502
- link rakuda_r3__upper_arm_cover_inside_r_1__ソリッド1: mass 6.71234e-06 -> 0.00706138
- link rakuda_r3__upper_arm_cover_inside_r_1__ソリッド1_1: mass 6.71234e-06 -> 0.00706138
- link rakuda_r3__waist_cover_hip_1__ソリッド1: mass 8.51661e-06 -> 0.00895947
- link rakuda_r3__x540_thrust_axk1160_1__ソリッド1: mass 5.48524e-06 -> 0.00577047
- link rakuda_r3__x540_thrust_axk1160_1__ソリッド1_1: mass 5.48524e-06 -> 0.00577047
- link x430_thrust_washer_1__part_1: mass 2.64406e-06 -> 0.00278155
- link x430_thrust_washer_1__part_1_1: mass 2.64406e-06 -> 0.00278155
- link x430_thrust_washer_1__part_1_2: mass 2.64406e-06 -> 0.00278155
- link x430_thrust_washer_1__part_1_3: mass 2.64406e-06 -> 0.00278155
- link x430_thrust_washer_1__part_1_4: mass 2.64406e-06 -> 0.00278155
- link xm430_w350_1__ソリッド2_11: mass 3.876e-08 -> 7.05432e-05
- link xm430_w350_1__ソリッド2_2: mass 3.876e-08 -> 7.05432e-05
- link xm430_w350_1__ソリッド2_3: mass 3.876e-08 -> 7.05432e-05
- link xm430_w350_1__ソリッド2_4: mass 3.876e-08 -> 7.05432e-05
- link xm430_w350_1__ソリッド2_5: mass 3.876e-08 -> 7.05432e-05
- link xm430_w350_1__ソリッド2_6: mass 3.876e-08 -> 7.05432e-05
- link xm430_w350_1__ソリッド2_7: mass 3.876e-08 -> 7.05432e-05
- link xm430_w350_1__ソリッド2_9: mass 3.876e-08 -> 7.05432e-05
- link xm430_w350_1__ソリッド3: mass 8.00924e-06 -> 0.0145757
- link xm430_w350_1__ソリッド3_1: mass 8.00924e-06 -> 0.0145768
- link xm430_w350_1__ソリッド3_10: mass 8.00924e-06 -> 0.0145768
- link xm430_w350_1__ソリッド3_11: mass 8.00924e-06 -> 0.0145768
- link xm430_w350_1__ソリッド3_2: mass 8.00924e-06 -> 0.0145768
- link xm430_w350_1__ソリッド3_3: mass 8.00924e-06 -> 0.0145768
- link xm430_w350_1__ソリッド3_4: mass 8.00924e-06 -> 0.0145768
- link xm430_w350_1__ソリッド3_5: mass 8.00924e-06 -> 0.0145768
- link xm430_w350_1__ソリッド3_6: mass 8.00924e-06 -> 0.0145768
- link xm430_w350_1__ソリッド3_7: mass 8.00924e-06 -> 0.0145768
- link xm430_w350_1__ソリッド3_8: mass 8.00924e-06 -> 0.0145768
- link xm430_w350_1__ソリッド3_9: mass 8.00924e-06 -> 0.0145768
- link xm430_w350_1__ソリッド4: mass 2.20536e-05 -> 0.0401343
- link xm430_w350_1__ソリッド4_1: mass 2.20536e-05 -> 0.0401375
- link xm430_w350_1__ソリッド4_10: mass 2.20536e-05 -> 0.0401375
- link xm430_w350_1__ソリッド4_11: mass 2.20536e-05 -> 0.0401375
- link xm430_w350_1__ソリッド4_2: mass 2.20536e-05 -> 0.0401375
- link xm430_w350_1__ソリッド4_3: mass 2.20536e-05 -> 0.0401375
- link xm430_w350_1__ソリッド4_4: mass 2.20536e-05 -> 0.0401375
- link xm430_w350_1__ソリッド4_5: mass 2.20536e-05 -> 0.0401375
- link xm430_w350_1__ソリッド4_6: mass 2.20536e-05 -> 0.0401375
- link xm430_w350_1__ソリッド4_7: mass 2.20536e-05 -> 0.0401375
- link xm430_w350_1__ソリッド4_8: mass 2.20536e-05 -> 0.0401375
- link xm430_w350_1__ソリッド4_9: mass 2.20536e-05 -> 0.0401375
- link xm430_w350_1__ソリッド5: mass 1.07968e-05 -> 0.0196486
- link xm430_w350_1__ソリッド5_1: mass 1.07968e-05 -> 0.0196502
- link xm430_w350_1__ソリッド5_10: mass 1.07968e-05 -> 0.0196502
- link xm430_w350_1__ソリッド5_11: mass 1.07968e-05 -> 0.0196502
- link xm430_w350_1__ソリッド5_2: mass 1.07968e-05 -> 0.0196502
- link xm430_w350_1__ソリッド5_3: mass 1.07968e-05 -> 0.0196502
- link xm430_w350_1__ソリッド5_4: mass 1.07968e-05 -> 0.0196502
- link xm430_w350_1__ソリッド5_5: mass 1.07968e-05 -> 0.0196502
- link xm430_w350_1__ソリッド5_6: mass 1.07968e-05 -> 0.0196502
- link xm430_w350_1__ソリッド5_7: mass 1.07968e-05 -> 0.0196502
- link xm430_w350_1__ソリッド5_8: mass 1.07968e-05 -> 0.0196502
- link xm430_w350_1__ソリッド5_9: mass 1.07968e-05 -> 0.0196502
- link xm540_w270_1__ソリッド2_2: mass 2.20928e-05 -> 0.0422856
- link xm540_w270_1__ソリッド2_3: mass 2.20928e-05 -> 0.0422856
- link xm540_w270_1__ソリッド2_4: mass 2.20928e-05 -> 0.0422856
- link xm540_w270_1__ソリッド4_1: mass 1.73735e-05 -> 0.0332444
- link xm540_w270_1__ソリッド4_1_2: mass 1.73735e-05 -> 0.0332529
- link xm540_w270_1__ソリッド4_1_4: mass 1.73735e-05 -> 0.0332529
- link xm540_w270_1__ソリッド4_2: mass 4.446e-08 -> 8.50964e-05
- link xm540_w270_1__ソリッド4_3: mass 4.446e-08 -> 8.50964e-05
- link xm540_w270_1__ソリッド4_4: mass 4.446e-08 -> 8.50964e-05
- link xm540_w270_1__ソリッド5_2: mass 4.04398e-05 -> 0.0774018
- link xm540_w270_1__ソリッド5_3: mass 4.04398e-05 -> 0.0774018
- link xm540_w270_1__ソリッド5_4: mass 4.04398e-05 -> 0.0774018

File: src/robopy/models/rakuda/assembly_2/urdf/assembly_2_convex_collision.urdf (robot description, URDF)
Before this commit: robot assembly_2, 153 links, 152 joints
Links:
- link _5シリーズ2列_nfs5_2040_297_1___nfs5_2040_910: mass 9.57636e-05 -> 0.258562
- link _ゴム足Φ24x10_c_30_rk_24_black_1__none_1: mass 3.25901e-06 -> 0.00358491
- link axk1106_1___axk1106: mass 1.52808e-06 -> 0.00168089
- link axk1106_1___axk1106_1: mass 1.52808e-06 -> 0.00412582
- link axk1106_1___axk1106_2: mass 1.52808e-06 -> 0.00412582
- link base_plate_03jk_rakuda_1__ソリッド1: mass 0.000712823 -> 5.59566
- link cable_guide_fr12_hinge_head_r4_1__ソリッド1: mass 2.66493e-06 -> 0.00280351
- link elbow_cover_right: mass 1.90245e-05 -> 0.0200138
- link fr12_h104_1__ソリッド1: mass 4.31461e-06 -> 0.0116495
- link fr12_h104_1__ソリッド1_1: mass 4.31461e-06 -> 0.0116495
- link fr12_h104_1__ソリッド1_2: mass 4.31461e-06 -> 0.0116495
- link fr12_h104_1__ソリッド1_3: mass 4.31461e-06 -> 0.0116495
- link fr12_h104_1__ソリッド1_4: mass 4.31461e-06 -> 0.0116495
- link fr12_s101_1__ソリッド1: mass 3.17353e-06 -> 0.00856853
- link fr12_s101_1__ソリッド1_1: mass 3.17353e-06 -> 0.00856853
- link fr12_s102_1__ソリッド1: mass 2.0777e-06 -> 0.00560978
- link fr12_s102_1__ソリッド1_1: mass 2.0777e-06 -> 0.00560978
- link fr13_h101_1__ソリッド1: mass 6.02982e-06 -> 0.0162805
- link fr13_h101_1__ソリッド1_1: mass 6.02982e-06 -> 0.0162805
- link hn12_i101_1__ソリッド1: mass 5.41761e-07 -> 0.00146275
- link hn12_i101_1__ソリッド1_1: mass 5.41761e-07 -> 0.00146275
- link hn12_i101_1__ソリッド1_2: mass 5.41761e-07 -> 0.00146275
- link hn12_i101_1__ソリッド1_3: mass 5.41761e-07 -> 0.00146275
- link hn12_i101_1__ソリッド1_4: mass 5.41761e-07 -> 0.00146275
- link hn12_n101_1__ソリッド1: mass 5.8065e-07 -> 0.00156776
- link hn12_n101_1__ソリッド1_1: mass 5.8065e-07 -> 0.00156776
- link hn12_n101_1__ソリッド1_2: mass 5.8065e-07 -> 0.00156776
- link hn12_n101_1__ソリッド1_3: mass 5.8065e-07 -> 0.00156776
- link hn12_n101_1__ソリッド1_4: mass 5.8065e-07 -> 0.00156776
- link hn12_n101_1__ソリッド1_5: mass 5.8065e-07 -> 0.00156776
- link hn12_n101_1__ソリッド1_6: mass 5.8065e-07 -> 0.00156776
- link hn12_n101_1__ソリッド1_7: mass 5.8065e-07 -> 0.00156776
- link hn12_n101_1__ソリッド1_8: mass 5.8065e-07 -> 0.00156776
- link hn12_n101_1__ソリッド1_9: mass 5.8065e-07 -> 0.00156776
- link hn13_c101_1__ソリッド1: mass 1.76909e-06 -> 0.00477655
- link hn13_c101_1__ソリッド1_1: mass 1.76909e-06 -> 0.00477655
- link hn13_c101_1__ソリッド1_2: mass 1.76909e-06 -> 0.00477655
- link hn13_i101_1__ソリッド1: mass 1.17425e-06 -> 0.00317047
- link hn13_i101_1__ソリッド1_1: mass 1.17425e-06 -> 0.00317047
- link hn13_n101_1__ソリッド1: mass 1.22568e-06 -> 0.00330934
- link hn13_n101_1__ソリッド1_1: mass 1.22568e-06 -> 0.00330934
- link igus_jfm_1113_05_1__1: mass 3.09557e-07 -> 0.000835805
- link igus_jfm_1113_05_1__1_1: mass 3.09557e-07 -> 0.000835805
- link igus_jfm_1113_05_1__1_2: mass 3.09557e-07 -> 0.000835805
- link igus_jfm_1113_05_1__1_3: mass 3.09557e-07 -> 0.000835805
- link intel_realsense_depth_camera_d435_1__ソリッド1_1: mass 3.65256e-05 -> 0.0465255
- link rakuda29_joint_upper_arm_r1_1__ソリッド1: mass 5.54227e-06 -> 0.00583046
- link rakuda29_joint_upper_arm_r1_1__ソリッド1_1: mass 5.54227e-06 -> 0.00583046
- link rakuda2_r3_waist_base_1__ソリッド1: mass 2.8514e-05 -> 0.0299967
- link rakuda34_r2__spacer_axk1160_waist_ring_r1_1__ソリッド1: mass 2.61695e-07 -> 0.000287864
- link rakuda34_r2__spacer_axk1160_waist_ring_r1_1__ソリッド1_1: mass 2.61695e-07 -> 0.000287864
- link rakuda_r3__arm_cover_elbow_r1_1__ソリッド1: mass 1.94674e-05 -> 0.0204797
- link rakuda_r3__arm_cover_upperarm_side_1__ソリッド1: mass 2.58744e-05 -> 0.0272199
- link rakuda_r3__arm_cover_upperarm_side_1__ソリッド1_1: mass 2.58744e-05 -> 0.0272199
- link rakuda_r3__arm_joint_upper_arm_back_1__ソリッド2: mass 4.29668e-06 -> 0.00452011
- link rakuda_r3__arm_joint_upper_arm_back_1__ソリッド2_1: mass 4.29668e-06 -> 0.00452011
- link rakuda_r3__base_cable_guide_d435usb_r1_1__ソリッド1: mass 3.18899e-06 -> 0.00335482
- link rakuda_r3__chest_cover_r1_1__ソリッド1: mass 1.28949e-05 -> 0.0135654
- link rakuda_r3__head_cable_guide_d435usb_1__ソリッド1: mass 4.08926e-07 -> 0.00043019
- link rakuda_r3__head_cover_front_1__ソリッド1: mass 1.06876e-05 -> 0.0112433
- link rakuda_r3__head_mount_d435_1__ソリッド1: mass 1.89546e-05 -> 0.0199402
- link rakuda_r3__neck_cable_guide2head_base_1__ソリッド1: mass 1.04854e-05 -> 0.0110306
- link rakuda_r3__neck_cover_r4_1__ソリッド1: mass 1.89252e-05 -> 0.0199093
- link rakuda_r3__plate_waist_x540_r8_1__ソリッド1: mass 9.67876e-05 -> 0.101821
- link rakuda_r3__shoulder_base_hinge_1__ソリッド1: mass 1.4263e-05 -> 0.0150046
- link rakuda_r3__shoulder_base_hinge_1__ソリッド1_1: mass 1.4263e-05 -> 0.0150046
- link rakuda_r3__shoulder_hinge_cover_1__ソリッド1: mass 7.08032e-06 -> 0.00744849
- link rakuda_r3__shoulder_hinge_cover_1__ソリッド1_2: mass 7.08032e-06 -> 0.00744849
- link rakuda_r3__spacer_axk1160_waist_r2_1__ソリッド1: mass 5.47367e-06 -> 0.0057583
- link rakuda_r3__upper_arm_cover_inside_l_1__ソリッド1: mass 6.71233e-06 -> 0.00706138
- link rakuda_r3__upper_arm_cover_inside_l_r1_1__ソリッド1: mass 6.89641e-06 -> 0.00725502
- link rakuda_r3__upper_arm_cover_inside_r_1__ソリッド1: mass 6.71234e-06 -> 0.00706138
- link rakuda_r3__upper_arm_cover_inside_r_1__ソリッド1_1: mass 6.71234e-06 -> 0.00706138
- link rakuda_r3__waist_cover_hip_1__ソリッド1: mass 8.51661e-06 -> 0.00895947
- link rakuda_r3__x540_thrust_axk1160_1__ソリッド1: mass 5.48524e-06 -> 0.00577047
- link rakuda_r3__x540_thrust_axk1160_1__ソリッド1_1: mass 5.48524e-06 -> 0.00577047
- link x430_thrust_washer_1__part_1: mass 2.64406e-06 -> 0.00278155
- link x430_thrust_washer_1__part_1_1: mass 2.64406e-06 -> 0.00278155
- link x430_thrust_washer_1__part_1_2: mass 2.64406e-06 -> 0.00278155
- link x430_thrust_washer_1__part_1_3: mass 2.64406e-06 -> 0.00278155
- link x430_thrust_washer_1__part_1_4: mass 2.64406e-06 -> 0.00278155
- link xm430_w350_1__ソリッド2_11: mass 3.876e-08 -> 7.05432e-05
- link xm430_w350_1__ソリッド2_2: mass 3.876e-08 -> 7.05432e-05
- link xm430_w350_1__ソリッド2_3: mass 3.876e-08 -> 7.05432e-05
- link xm430_w350_1__ソリッド2_4: mass 3.876e-08 -> 7.05432e-05
- link xm430_w350_1__ソリッド2_5: mass 3.876e-08 -> 7.05432e-05
- link xm430_w350_1__ソリッド2_6: mass 3.876e-08 -> 7.05432e-05
- link xm430_w350_1__ソリッド2_7: mass 3.876e-08 -> 7.05432e-05
- link xm430_w350_1__ソリッド2_9: mass 3.876e-08 -> 7.05432e-05
- link xm430_w350_1__ソリッド3: mass 8.00924e-06 -> 0.0145757
- link xm430_w350_1__ソリッド3_1: mass 8.00924e-06 -> 0.0145768
- link xm430_w350_1__ソリッド3_10: mass 8.00924e-06 -> 0.0145768
- link xm430_w350_1__ソリッド3_11: mass 8.00924e-06 -> 0.0145768
- link xm430_w350_1__ソリッド3_2: mass 8.00924e-06 -> 0.0145768
- link xm430_w350_1__ソリッド3_3: mass 8.00924e-06 -> 0.0145768
- link xm430_w350_1__ソリッド3_4: mass 8.00924e-06 -> 0.0145768
- link xm430_w350_1__ソリッド3_5: mass 8.00924e-06 -> 0.0145768
- link xm430_w350_1__ソリッド3_6: mass 8.00924e-06 -> 0.0145768
- link xm430_w350_1__ソリッド3_7: mass 8.00924e-06 -> 0.0145768
- link xm430_w350_1__ソリッド3_8: mass 8.00924e-06 -> 0.0145768
- link xm430_w350_1__ソリッド3_9: mass 8.00924e-06 -> 0.0145768
- link xm430_w350_1__ソリッド4: mass 2.20536e-05 -> 0.0401343
- link xm430_w350_1__ソリッド4_1: mass 2.20536e-05 -> 0.0401375
- link xm430_w350_1__ソリッド4_10: mass 2.20536e-05 -> 0.0401375
- link xm430_w350_1__ソリッド4_11: mass 2.20536e-05 -> 0.0401375
- link xm430_w350_1__ソリッド4_2: mass 2.20536e-05 -> 0.0401375
- link xm430_w350_1__ソリッド4_3: mass 2.20536e-05 -> 0.0401375
- link xm430_w350_1__ソリッド4_4: mass 2.20536e-05 -> 0.0401375
- link xm430_w350_1__ソリッド4_5: mass 2.20536e-05 -> 0.0401375
- link xm430_w350_1__ソリッド4_6: mass 2.20536e-05 -> 0.0401375
- link xm430_w350_1__ソリッド4_7: mass 2.20536e-05 -> 0.0401375
- link xm430_w350_1__ソリッド4_8: mass 2.20536e-05 -> 0.0401375
- link xm430_w350_1__ソリッド4_9: mass 2.20536e-05 -> 0.0401375
- link xm430_w350_1__ソリッド5: mass 1.07968e-05 -> 0.0196486
- link xm430_w350_1__ソリッド5_1: mass 1.07968e-05 -> 0.0196502
- link xm430_w350_1__ソリッド5_10: mass 1.07968e-05 -> 0.0196502
- link xm430_w350_1__ソリッド5_11: mass 1.07968e-05 -> 0.0196502
- link xm430_w350_1__ソリッド5_2: mass 1.07968e-05 -> 0.0196502
- link xm430_w350_1__ソリッド5_3: mass 1.07968e-05 -> 0.0196502
- link xm430_w350_1__ソリッド5_4: mass 1.07968e-05 -> 0.0196502
- link xm430_w350_1__ソリッド5_5: mass 1.07968e-05 -> 0.0196502
- link xm430_w350_1__ソリッド5_6: mass 1.07968e-05 -> 0.0196502
- link xm430_w350_1__ソリッド5_7: mass 1.07968e-05 -> 0.0196502
- link xm430_w350_1__ソリッド5_8: mass 1.07968e-05 -> 0.0196502
- link xm430_w350_1__ソリッド5_9: mass 1.07968e-05 -> 0.0196502
- link xm540_w270_1__ソリッド2_2: mass 2.20928e-05 -> 0.0422856
- link xm540_w270_1__ソリッド2_3: mass 2.20928e-05 -> 0.0422856
- link xm540_w270_1__ソリッド2_4: mass 2.20928e-05 -> 0.0422856
- link xm540_w270_1__ソリッド4_1: mass 1.73735e-05 -> 0.0332444
- link xm540_w270_1__ソリッド4_1_2: mass 1.73735e-05 -> 0.0332529
- link xm540_w270_1__ソリッド4_1_4: mass 1.73735e-05 -> 0.0332529
- link xm540_w270_1__ソリッド4_2: mass 4.446e-08 -> 8.50964e-05
- link xm540_w270_1__ソリッド4_3: mass 4.446e-08 -> 8.50964e-05
- link xm540_w270_1__ソリッド4_4: mass 4.446e-08 -> 8.50964e-05
- link xm540_w270_1__ソリッド5_2: mass 4.04398e-05 -> 0.0774018
- link xm540_w270_1__ソリッド5_3: mass 4.04398e-05 -> 0.0774018
- link xm540_w270_1__ソリッド5_4: mass 4.04398e-05 -> 0.0774018
